File: ESP8285-Miniboard/esp8285-miniboard-v1.0.sch (EAGLE design)
At the start: 40 parts, among them Q1 FA-128

Commit message: Another Rev 1.0
Connections:
- net N$IO1: now also PROG.2
- net N$IO2: no longer PROG.2
Other:
- moved on the sheet: D2, R8
Changed lines of the file:
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@@
 <attribute name="VALUE" x="91.44" y="163.576" size="1.778" layer="96" rot="R180"/>
 </instance>
-<instance part="D2" gate="G$1" x="106.68" y="143.51" rot="R270"/>
-<instance part="R8" gate="G$1" x="106.68" y="153.67" rot="R90"/>
-<instance part="GND13" gate="1" x="106.68" y="137.16"/>
+<instance part="D2" gate="G$1" x="177.8" y="138.43" rot="R270"/>
+<instance part="R8" gate="G$1" x="177.8" y="148.59" rot="R90"/>
+<instance part="GND13" gate="1" x="177.8" y="132.08"/>
 </instances>
 <busses>
@@
 </segment>
 </net>
-<net name="N$IO2" class="0">
-<segment>
-<wire x1="160.02" y1="99.06" x2="185.42" y2="99.06" width="0.1524" layer="91"/>
-<pinref part="PROG" gate="G$1" pin="2"/>
-<pinref part="U$1" gate="G$1" pin="TX1-2"/>
-<pinref part="2" gate="G$1" pin="1"/>
-<wire x1="162.56" y1="119.38" x2="160.02" y2="119.38" width="0.1524" layer="91"/>
-<wire x1="160.02" y1="119.38" x2="142.24" y2="119.38" width="0.1524" layer="91"/>
-<wire x1="160.02" y1="99.06" x2="160.02" y2="119.38" width="0.1524" layer="91"/>
-<junction x="160.02" y="119.38"/>
-</segment>
-</net>
 <net name="N$IO3" class="0">
 <segment>
@@
 <pinref part="D2" gate="G$1" pin="+"/>
 <pinref part="R8" gate="G$1" pin="1"/>
-<wire x1="106.68" y1="149.86" x2="106.68" y2="147.32" width="0.1524" layer="91"/>
+<wire x1="177.8" y1="144.78" x2="177.8" y2="142.24" width="0.1524" layer="91"/>
+</segment>
+</net>
+<net name="N$IO2" class="0">
+<segment>
+<pinref part="U$1" gate="G$1" pin="TX1-2"/>
+<pinref part="2" gate="G$1" pin="1"/>
+<wire x1="162.56" y1="119.38" x2="142.24" y2="119.38" width="0.1524" layer="91"/>
 </segment>
 </net>
 <net name="N$IO1" class="0">
 <segment>
-<wire x1="106.68" y1="160.02" x2="106.68" y2="157.48" width="0.1524" layer="91"/>
+<wire x1="160.02" y1="99.06" x2="185.42" y2="99.06" width="0.1524" layer="91"/>
+<pinref part="PROG" gate="G$1" pin="2"/>
+<wire x1="177.8" y1="154.94" x2="177.8" y2="152.4" width="0.1524" layer="91"/>
 <pinref part="R8" gate="G$1" pin="2"/>
 <pinref part="1" gate="G$1" pin="1"/>
 <pinref part="U$1" gate="G$1" pin="TX0-1"/>
-<wire x1="162.56" y1="121.92" x2="144.78" y2="121.92" width="0.1524" layer="91"/>
-<wire x1="144.78" y1="121.92" x2="142.24" y2="121.92" width="0.1524" layer="91"/>
-<wire x1="106.68" y1="160.02" x2="144.78" y2="160.02" width="0.1524" layer="91"/>
-<wire x1="144.78" y1="160.02" x2="144.78" y2="121.92" width="0.1524" layer="91"/>
-<junction x="144.78" y="121.92"/>
-</segment>
-</net>
+<wire x1="162.56" y1="121.92" x2="160.02" y2="121.92" width="0.1524" layer="91"/>
+<wire x1="160.02" y1="121.92" x2="142.24" y2="121.92" width="0.1524" layer="91"/>
+<wire x1="177.8" y1="154.94" x2="160.02" y2="154.94" width="0.1524" layer="91"/>
+<wire x1="160.02" y1="154.94" x2="160.02" y2="121.92" width="0.1524" layer="91"/>
+<junction x="160.02" y="121.92"/>
+<wire x1="160.02" y1="99.06" x2="160.02" y2="121.92" width="0.1524" layer="91"/>
+<junction x="160.02" y="121.92"/>
+</segment>
+</net>

Commit message: Hopefully final V1.0
Parts:
- added CH_PU: (no value), Ma-ESP8285:TESTPIN-1X1-SM
Connections:
- net N$CHIP_PU: now also CH_PU.1
Other:
- note added: "Blue Tx LED"
- note added: "Essential pins for programming and running VDD pins = +3.3V (3.0-3.6V) CH_PD = H (10k pull-up) IO15 = L (10k pull-down) Tx0-IO1 = To Rx of programmer Rx0-IO3 = To Tx of programmer IO0 = To programmer (Nodemcu circuit) Reset = To programmer (Nodemcu circuit)"
- note added: "For deep sleep"
- note added: "GPIO0"
- note added: "Programming connector"
- note added: "RX->TX"
- note added: "Red Power LED"
- note added: "Reset"
- note added: "TX->RX"
- note removed: "DTR"
- note removed: "Programming pinout ESP8285 = Serial Tx-IO2 = Rx Rx = Tx IO0 = DTR IO15 = H CH_PD = H Reset = RTS"
- note removed: "RTS"
- note removed: "RX"
- note removed: "TX"
- moved on the sheet: GND, R2

Commit message: Final v1.0 fixed silkscreen, added testpoint, reduced via size
Parts:
- removed TOUT: (no value), Ma-ESP8285:TESTPIN-1X1-SM
- added R9: 10K, Seeed-OPL-Resistor:SMD-RES-10K-1%-1/10W(0603)
- added TO: (no value), Markus:TESTPIN-1X1-SM
- 0, 1, 10, 11, 12, 13, 14, 15, 16, 2, 3, 3V3, 4, 5, 6, 7, 8, 9, CH_PU, GND, VDDRTC: device Ma-ESP8285:TESTPIN-1X1-SM -> Markus:TESTPIN-1X1-SM
Connections:
- net +3V3: now also R9.2
- net N$IO2: now also R9.1
- net N$TOUT: now also TO.1; no longer TOUT.1
Changed lines of the file:
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@@
 <part name="R3" library="Seeed-OPL-Resistor" deviceset="SMD-RES-10K-1%-1/10W(0603)" device="" value="10K"/>
 <part name="+3V3" library="supply1" deviceset="+3V3" device=""/>
-<part name="15" library="Ma-ESP8285" deviceset="TESTPIN-1X1-SM" device=""/>
-<part name="14" library="Ma-ESP8285" deviceset="TESTPIN-1X1-SM" device=""/>
-<part name="13" library="Ma-ESP8285" deviceset="TESTPIN-1X1-SM" device=""/>
-<part name="16" library="Ma-ESP8285" deviceset="TESTPIN-1X1-SM" device=""/>
-<part name="12" library="Ma-ESP8285" deviceset="TESTPIN-1X1-SM" device=""/>
-<part name="11" library="Ma-ESP8285" deviceset="TESTPIN-1X1-SM" device=""/>
-<part name="10" library="Ma-ESP8285" deviceset="TESTPIN-1X1-SM" device=""/>
-<part name="9" library="Ma-ESP8285" deviceset="TESTPIN-1X1-SM" device=""/>
-<part name="8" library="Ma-ESP8285" deviceset="TESTPIN-1X1-SM" device=""/>
-<part name="7" library="Ma-ESP8285" deviceset="TESTPIN-1X1-SM" device=""/>
-<part name="6" library="Ma-ESP8285" deviceset="TESTPIN-1X1-SM" device=""/>
-<part name="5" library="Ma-ESP8285" deviceset="TESTPIN-1X1-SM" device=""/>
-<part name="4" library="Ma-ESP8285" deviceset="TESTPIN-1X1-SM" device=""/>
-<part name="3" library="Ma-ESP8285" deviceset="TESTPIN-1X1-SM" device=""/>
-<part name="2" library="Ma-ESP8285" deviceset="TESTPIN-1X1-SM" device=""/>
-<part name="0" library="Ma-ESP8285" deviceset="TESTPIN-1X1-SM" device=""/>
-<part name="1" library="Ma-ESP8285" deviceset="TESTPIN-1X1-SM" device=""/>
+<part name="15" library="Markus" deviceset="TESTPIN-1X1-SM" device=""/>
+<part name="14" library="Markus" deviceset="TESTPIN-1X1-SM" device=""/>
+<part name="13" library="Markus" deviceset="TESTPIN-1X1-SM" device=""/>
+<part name="16" library="Markus" deviceset="TESTPIN-1X1-SM" device=""/>
+<part name="12" library="Markus" deviceset="TESTPIN-1X1-SM" device=""/>
+<part name="11" library="Markus" deviceset="TESTPIN-1X1-SM" device=""/>
+<part name="10" library="Markus" deviceset="TESTPIN-1X1-SM" device=""/>
+<part name="9" library="Markus" deviceset="TESTPIN-1X1-SM" device=""/>
+<part name="8" library="Markus" deviceset="TESTPIN-1X1-SM" device=""/>
+<part name="7" library="Markus" deviceset="TESTPIN-1X1-SM" device=""/>
+<part name="6" library="Markus" deviceset="TESTPIN-1X1-SM" device=""/>
+<part name="5" library="Markus" deviceset="TESTPIN-1X1-SM" device=""/>
+<part name="4" library="Markus" deviceset="TESTPIN-1X1-SM" device=""/>
+<part name="3" library="Markus" deviceset="TESTPIN-1X1-SM" device=""/>
+<part name="2" library="Markus" deviceset="TESTPIN-1X1-SM" device=""/>
+<part name="0" library="Markus" deviceset="TESTPIN-1X1-SM" device=""/>
+<part name="1" library="Markus" deviceset="TESTPIN-1X1-SM" device=""/>
 <part name="GND9" library="supply1" deviceset="GND" device=""/>
 <part name="+3V4" library="supply1" deviceset="+3V3" device=""/>
 <part name="C5" library="Seeed-OPL-Capacitor" deviceset="CERAMIC-10UF-6.3V-20%-X5R(0603)" device="" value="10UF 6.3V"/>
 <part name="GND10" library="supply1" deviceset="GND" device=""/>
-<part name="TOUT" library="Ma-ESP8285" deviceset="TESTPIN-1X1-SM" device=""/>
+<part name="TO" library="Markus" deviceset="TESTPIN-1X1-SM" device=""/>
 <part name="R4" library="Seeed-OPL-Resistor" deviceset="SMD-RES-0R-5%-1/10W(0603)" device="" value="0R"/>
 <part name="R5" library="Seeed-OPL-Resistor" deviceset="SMD-RES-10K-1%-1/10W(0603)" device="" value="10K"/>
 <part name="R6" library="Seeed-OPL-Resistor" deviceset="SMD-RES-10K-1%-1/10W(0603)" device="" value="10K"/>
 <part name="GND12" library="supply1" deviceset="GND" device=""/>
-<part name="VDDRTC" library="Ma-ESP8285" deviceset="TESTPIN-1X1-SM" device=""/>
-<part name="3V3" library="Ma-ESP8285" deviceset="TESTPIN-1X1-SM" device=""/>
-<part name="GND" library="Ma-ESP8285" deviceset="TESTPIN-1X1-SM" device=""/>
+<part name="VDDRTC" library="Markus" deviceset="TESTPIN-1X1-SM" device=""/>
+<part name="3V3" library="Markus" deviceset="TESTPIN-1X1-SM" device=""/>
+<part name="GND" library="Markus" deviceset="TESTPIN-1X1-SM" device=""/>
 <part name="D1" library="Seeed-OPL-Diode" deviceset="SMD-LED-CLEAR-RED(0805)" device="" value="RED-0805"/>
 <part name="R7" library="Seeed-OPL-Resistor" deviceset="SMD-RES-330R-1%-1/10W(0603)" device="" value="330R"/>
@@
 <part name="R8" library="Seeed-OPL-Resistor" deviceset="SMD-RES-330R-1%-1/10W(0603)" device="" value="330R"/>
 <part name="GND13" library="supply1" deviceset="GND" device=""/>
-<part name="CH_PU" library="Ma-ESP8285" deviceset="TESTPIN-1X1-SM" device=""/>
+<part name="CH_PU" library="Markus" deviceset="TESTPIN-1X1-SM" device=""/>
+<part name="+3V6" library="supply1" deviceset="+3V3" device=""/>
+<part name="R9" library="Seeed-OPL-Resistor" deviceset="SMD-RES-10K-1%-1/10W(0603)" device="" value="10K"/>
 </parts>
 <sheets>
@@
 </instance>
 <instance part="GND10" gate="1" x="68.58" y="111.76"/>
-<instance part="TOUT" gate="G$1" x="96.52" y="88.9" smashed="yes" rot="R90">
+<instance part="TO" gate="G$1" x="96.52" y="88.9" smashed="yes" rot="R90">
 <attribute name="NAME" x="98.806" y="90.805" size="1.27" layer="95" rot="R180"/>
 <attribute name="VALUE" x="102.87" y="85.09" size="1.778" layer="96" rot="R90"/>
@@
 <attribute name="NAME" x="86.106" y="85.725" size="1.27" layer="95" rot="R180"/>
 <attribute name="VALUE" x="90.17" y="80.01" size="1.778" layer="96" rot="R90"/>
+</instance>
+<instance part="+3V6" gate="G$1" x="147.32" y="142.24" smashed="yes">
+<attribute name="VALUE" x="149.86" y="145.796" size="1.778" layer="96" rot="R180"/>
+</instance>
+<instance part="R9" gate="G$1" x="147.32" y="132.08" smashed="yes" rot="R90">
+<attribute name="NAME" x="145.3134" y="130.556" size="1.778" layer="95" rot="R90"/>
+<attribute name="VALUE" x="151.13" y="130.302" size="1.778" layer="96" rot="R90"/>
 </instance>
 </instances>
@@
 <pinref part="+3V5" gate="G$1" pin="+3V3"/>
 </segment>
+<segment>
+<pinref part="+3V6" gate="G$1" pin="+3V3"/>
+<pinref part="R9" gate="G$1" pin="2"/>
+<wire x1="147.32" y1="139.7" x2="147.32" y2="135.89" width="0.1524" layer="91"/>
+</segment>
 </net>
 <net name="N$XTAL-IN" class="0">
@@
 <segment>
 <pinref part="U$1" gate="G$1" pin="TOUT"/>
-<pinref part="TOUT" gate="G$1" pin="1"/>
+<pinref part="TO" gate="G$1" pin="1"/>
 <wire x1="99.06" y1="88.9" x2="104.14" y2="88.9" width="0.1524" layer="91"/>
 </segment>
@@
 <pinref part="U$1" gate="G$1" pin="TX1-2"/>
 <pinref part="2" gate="G$1" pin="1"/>
-<wire x1="162.56" y1="119.38" x2="142.24" y2="119.38" width="0.1524" layer="91"/>
-</segment>
-</net>
+<wire x1="162.56" y1="119.38" x2="147.32" y2="119.38" width="0.1524" layer="91"/>
+<pinref part="R9" gate="G$1" pin="1"/>
+<wire x1="147.32" y1="119.38" x2="142.24" y2="119.38" width="0.1524" layer="91"/>
+<wire x1="147.32" y1="128.27" x2="147.32" y2="119.38" width="0.1524" layer="91"/>
+<junction x="147.32" y="119.38"/>
+</segment>
+</net>
